Commit message: drivers and robots packages cleanup

File: robots/ros2/utias_grizzly_description/urdf/accessories/sensor_mast.urdf.xacro (robot description, xacro)
@@ -25,5 +25,5 @@
 This program contains the description of the robot base model for the Clearpath Grizzly
 -->
-<robot xmlns:xacro="http://ros.org/wiki/xacro" name="asrl__grizzly">
+<robot xmlns:xacro="http://ros.org/wiki/xacro" name="utias_grizzly_description">
   <joint name="sensor_mast_joint"
          type="fixed">
@@ -48,5 +48,5 @@
               rpy="0 0 0" />
       <geometry>
-        <mesh filename="package://asrl__grizzly/mesh/sensor_mast.stl" />
+        <mesh filename="package://utias_grizzly_description/mesh/sensor_mast.stl" />
       </geometry>
       <material name="Black" />
